File: electronics/audio-amplifier.kicad_pcb (KiCad board)
At the start: 2 copper layers, 88.8 x 54 mm, 55 parts, among them J1 AUDIO-JACK, J3 AUDIO-JACK, J4 ECS00108, P2 HEADER-GENERIC-2WAY, P3 HEADER-GENERIC-2WAY, Q1 ECS00110, SW1 DPDT-GENERIC, U1 ECS00104

Commit message: Uploading completed design files.
Parts:
- R12: value DUAL-POT -> ECS00238; footprint ECFootprints:DUAL-POT2 -> ECFootprints:ECS00238F
- SW1: value DPDT-GENERIC -> ECS00237; footprint ECFootprints:DPDT-GENERIC -> ECFootprints:ECS00237F
- moved TP9 79.5 mm to (77.0, 40.5)
- moved SW1 70.9 mm to (50.0, 68.2)
- moved R12 70.0 mm to (58.5, 68.2), turned to 0 degrees
- moved TP1 68.5 mm to (62.8, 61.0)
- moved NT1 68.0 mm to (86.8, 82.7)
- moved U1 68.0 mm to (80.0, 63.8)
- moved C1 68.0 mm to (49.8, 54.8)
- moved C10 68.0 mm to (107.0, 64.8)
- moved C11 68.0 mm to (76.8, 81.0)
- moved C12 68.0 mm to (107.0, 54.2)
- moved C13 68.0 mm to (107.0, 71.2)
- moved C14 68.0 mm to (77.0, 46.0)
- moved C15 68.0 mm to (88.2, 52.5)
- moved C16 68.0 mm to (88.2, 73.0)
- moved C17 68.0 mm to (68.2, 72.5)
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Connections:
- SW1 pad 2: Net-(R12-Pad3B) -> Net-(R12-Pad6)
- SW1 pad 5: Net-(R12-Pad3A) -> Net-(R12-Pad3)
- TP9 pad 1: GNDA -> GND
Routing:
- net Net-(R12-Pad6): track 0.00 -> 41.8 mm
- net /CH2_R: track 11.8 -> 26.6 mm
- net Net-(R12-Pad3): track 0.00 -> 12.3 mm
- net /AUDIO_IN_L: track 10.2 -> 21.1 mm
- net Net-(R12-Pad3A): track 9.96 -> 0.00 mm
- net Net-(R12-Pad3B): track 6.78 -> 0.00 mm
- net /CH1_L: track 15.3 -> 8.97 mm
- net /CH2_L: track 16.3 -> 11.4 mm
- net GNDA: track 11.2 -> 14.5 mm, vias 0 -> 2
- net GND: track 25.2 -> 28.4 mm
- net /AUDIO_IN_R: track 13.7 -> 10.8 mm
Other:
- net class Default: trace_width 0.2 -> 0.5
- net class PWR: clearance 0.5 -> 0.2; trace_width 0.2 -> 0.5
- board text added: "0.20 MM 0.20 MM 0.20 MM 3.50 MM"
- board text added: "0.50 MM 1.50 MM 0.20 MM 0.60 MM 0.50 MM"
- board text added: "1. FABRICATE PER ANSI/IPC-1-600, IPC-QE-605, IPC-4101, IPC-4552 AND IPC-SM-840 SPECIFICATIONS. MUST USE ROHS-COMPLIANT MATERIALS. 2. MATERIAL: BASE MATERIAL LAMINATED EPOXY GLASS FR-4, NOM .062”, COLOUR NATURAL. NOM 1 OZ COPER WEIGHT. THICKNESS .070” MAX AFTER PLATING AND FINISHING. PREFER ROHS COMPLIANT PER IPC-4101 SLASH SHEETS #26 OR #83 OR #98 WITH MINIMUM TG 135 DEGREE C OR HIGHER, TD 300 DE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"
- board text added: "1.6 MM +/- 0.1 MM"
- board text added: "B-STAGE (0.33 MM REF)"
- board text added: "BOT LAYER"
- board text added: "COMPONENT SIDE"
- board text added: "FR4 EPOXY"
- board text added: "GENERAL NOTES"
- board text added: "LAYER DETAIL"
- board text added: "SOLDERMASK BOTTOM"
- board text added: "SOLDERMASK TOP"
- board text added: "TOP LAYER (VOLTAGE/RTN SIGNAL TRACES)"
- board text added: "TRACE WIDTH; ANULUS HOLE-TO-HOLE SILKSCREEN LINE MINIMUM HOLE SIZE (PLATED) BOARD EDGE-TO-COPPER"
- board text added: "TRACE-TO-TRACE; TRACE-TO-PAD PAD-TO-PAD SILKSCREEN-TO-BARE COPPER MAXIMUM HOLE SIZE (UNPLATED)"
