File: electronics/audio-amplifier.sch (KiCad schematic (older format))
At the start: 55 parts, among them J1 AUDIO-JACK, J3 AUDIO-JACK, J4 ECS00108, P2 HEADER-GENERIC-2WAY, P3 HEADER-GENERIC-2WAY, Q1 ECS00110, SW1 DPDT-GENERIC, U1 ECS00104

Commit message: Uploading completed design files.
Parts:
- removed R12: DUAL-POT, ECFootprints:DUAL-POT2, symbol Resistors:DUAL-POT
- removed SW1: DPDT-GENERIC, ECFootprints:DPDT-GENERIC, symbol Misc:DPDT-GENERIC
- added R12: ECS00238, ECFootprints:ECS00238F, symbol Resistors:ECS00238
- added SW1: ECS00237, ECFootprints:ECS00237F, symbol Switches:ECS00237
Connections:
- net AUDIO_IN_L: now also R12.5
- net AUDIO_IN_R: now also R12.2
- net CH1_L: now also SW1.1
- net CH1_R: now also SW1.4
- net CH2_L: now also SW1.3
- net CH2_R: now also SW1.6
- net GND: now also TP9.1
- net GNDA: now also R12.1, R12.4; no longer TP9.1
- new net: R12.6, SW1.2
- new net: R12.3, SW1.5
Other:
- moved on the sheet: C10, C12, C13, C9, L1, L2, P2, P3, R10, R11, TP6, TP7
